File: CAN_pitot.kicad_sch (KiCad schematic)
At the start: 20 parts, among them J1 SM04B-GHS-TB(LF)(SN)-, J2 SM04B-GHS-TB(LF)(SN)-, J3 SM04B-GHS-TB(LF)(SN)-, U1 NCV8705MT33TCG, U2 LM66100DCKR, U3 TJA1051TK/3,118

Commit message: More parts
Changed lines of the file:
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@@
     (effects (font (size 1 1)) (justify left bottom))
+  )
+  (label "Transistor" (at 118.11 74.93 0)
+    (effects (font (size 3 3)) (justify left bottom))
   )
   (label "CAN_P" (at 201.93 63.5 0)
@@
       (effects (font (size 1 1)) (justify right) hide)
     )
-  )
-  (hierarchical_label "First" (shape input) (at 16.51 191.77 0)
-    (effects (font (size 5 5)) (justify left))
   )
   (symbol (lib_id "3-1879460-1:3-1879460-1") (at 41.91 124.46 90) (unit 1)
@@
       (reference "#PWR0107") (unit 1) (value "+5V") (footprint "")
     )
+    (path "/82810f7f-9499-4602-9be8-4cf6e7e02f75/9753a417-ebdd-4926-b843-29c9ee0995cc"
+      (reference "#PWR0108") (unit 1) (value "GND") (footprint "")
+    )
+    (path "/82810f7f-9499-4602-9be8-4cf6e7e02f75/4345867c-fbdb-4544-9393-c738ce29cf5f"
+      (reference "#PWR0109") (unit 1) (value "GND") (footprint "")
+    )
+    (path "/82810f7f-9499-4602-9be8-4cf6e7e02f75/8d79923b-1390-462f-aa5f-12627d6194eb"
+      (reference "#PWR0110") (unit 1) (value "3.3V") (footprint "")
+    )
+    (path "/82810f7f-9499-4602-9be8-4cf6e7e02f75/1e139b0a-5e9f-49de-83bd-32d90b66d278"
+      (reference "#PWR0111") (unit 1) (value "GND") (footprint "")
+    )
+    (path "/82810f7f-9499-4602-9be8-4cf6e7e02f75/d6a1068c-da60-4f26-b272-a69dba6b0940"
+      (reference "#PWR0112") (unit 1) (value "3.3V") (footprint "")
+    )
+    (path "/82810f7f-9499-4602-9be8-4cf6e7e02f75/7437f239-4b0b-4b0e-a081-4180de20ebc2"
+      (reference "#PWR0113") (unit 1) (value "+5V") (footprint "")
+    )
     (path "/47f1a27e-e9c3-44f7-a95c-11c2c1def436"
       (reference "C1") (unit 1) (value "10uF") (footprint "SnapEDA Library:CAPC1608X90")
@@
       (reference "C13") (unit 1) (value "2.2uF") (footprint "SnapEDA Library:CAPC1608X90")
     )
+    (path "/82810f7f-9499-4602-9be8-4cf6e7e02f75/26fb6109-f9a1-483e-8722-892e6718f577"
+      (reference "C14") (unit 1) (value "2.2uF") (footprint "SnapEDA Library:CAPC1608X90")
+    )
+    (path "/82810f7f-9499-4602-9be8-4cf6e7e02f75/eaeec0d6-feba-4690-bcee-7efc21cd0ff1"
+      (reference "C15") (unit 1) (value "2.2uF") (footprint "SnapEDA Library:CAPC1608X90")
+    )
     (path "/4c5a3b26-c5fc-4ec8-a374-a75a1e8f35d3"
       (reference "D1") (unit 1) (value "SMBJ64") (footprint "DIOM4336X265N")
@@
       (reference "D6") (unit 1) (value "SMBJ64") (footprint "DIOM4336X265N")
     )
+    (path "/82810f7f-9499-4602-9be8-4cf6e7e02f75/a4028201-e5d9-4295-bc53-219ba530d00a"
+      (reference "D7") (unit 1) (value "Red") (footprint "LED_SML-D12FWT86")
+    )
+    (path "/82810f7f-9499-4602-9be8-4cf6e7e02f75/e482747f-28b1-4a46-927a-2f5fed51ad9a"
+      (reference "D8") (unit 1) (value "Green") (footprint "LED_SML-D12FWT86")
+    )
+    (path "/82810f7f-9499-4602-9be8-4cf6e7e02f75/ba740146-b83f-4add-a1ee-73c426cec79f"
+      (reference "D9") (unit 1) (value "Blue") (footprint "LED_SML-D12FWT86")
+    )
     (path "/753a45f8-7ceb-49d3-9e29-ecbeec71d768"
       (reference "J1") (unit 1) (value "SM04B-GHS-TB(LF)(SN)-") (footprint "SnapEDA Library:JST_SM04B-GHS-TB(LF)(SN)-")
@@
       (reference "R4") (unit 1) (value "1.5K") (footprint "SnapEDA Library:RESC1608X50N")
     )
+    (path "/82810f7f-9499-4602-9be8-4cf6e7e02f75/bd0a8cf3-b21d-46f9-a4d0-37c36563309b"
+      (reference "R5") (unit 1) (value "100K") (footprint "SnapEDA Library:RESC1608X50N")
+    )
+    (path "/82810f7f-9499-4602-9be8-4cf6e7e02f75/885a4139-562f-4301-8752-db9752677d13"
+      (reference "R6") (unit 1) (value "100K") (footprint "SnapEDA Library:RESC1608X50N")
+    )
+    (path "/82810f7f-9499-4602-9be8-4cf6e7e02f75/d0596217-ae78-47dc-8420-fc23415e4030"
+      (reference "R7") (unit 1) (value "604") (footprint "SnapEDA Library:RESC1608X50N")
+    )
+    (path "/82810f7f-9499-4602-9be8-4cf6e7e02f75/961028c6-4ba3-4ed3-a07c-a5d4c5581dd1"
+      (reference "R8") (unit 1) (value "604") (footprint "SnapEDA Library:RESC1608X50N")
+    )
+    (path "/82810f7f-9499-4602-9be8-4cf6e7e02f75/c64fe9d9-289d-4d12-b123-e918e145e6fe"
+      (reference "R9") (unit 1) (value "330") (footprint "SnapEDA Library:RESC1608X50N")
+    )
     (path "/65040185-1a42-4313-8d55-eb71a9980d5a"
