File: untitled.kicad_sch (KiCad schematic)
At the start: 11 parts, among them J4 SM06B-SRSS-TB(LF)(SN), U4 STM32F412CGUx

Commit message: More parts
Parts:
- added C14, C15: 2.2uF, SnapEDA Library:CAPC1608X90, symbol LD03YC101KAB2A:LD03YC101KAB2A
- added D7: Red, LED_SML-D12FWT86, symbol SML-D12FWT86:SML-D12FWT86
- added D8: Green, LED_SML-D12FWT86, symbol SML-D12FWT86:SML-D12FWT86
- added D9: Blue, LED_SML-D12FWT86, symbol SML-D12FWT86:SML-D12FWT86
- added R5, R6: 100K, SnapEDA Library:RESC1608X50N, symbol 3-1879460-1:3-1879460-1
- added R7, R8: 604, SnapEDA Library:RESC1608X50N, symbol 3-1879460-1:3-1879460-1
- added R9: 330, SnapEDA Library:RESC1608X50N, symbol 3-1879460-1:3-1879460-1
Connections:
- net +5V: now also U4.9 (VDDA), C15.1, D7.A, D8.A, D9.A, R6.2
- net GNDREF: now also U4.8 (VSSA), C14.2, C15.2, R5.1
- net LED_TIM1_CH1_RED: now also R7.1
- net LED_TIM1_CH2_GREEN: now also R8.1
- net LED_TIM1_CH3_BLUE: now also R9.1
- net at U4.22 (VCAP_1): now also C14.1
- net at U4.44 (BOOT0): now also R5.2
- net OSCILLATOR: now reaches U4.5 (PH0)
- net at U4.7 (NRST): now also R6.1
- new net: D8.C, R8.2
- new net: D7.C, R7.2
- new net: D9.C, R9.2
- no-connect marks 22 -> 23
